Commit message: [fix]modified details

File: model/urdf/hexa_leg.xacro (robot description, xacro)
@@ -104,4 +104,32 @@
             </geometry>
             </collision>
+            <!-- 座標系確認用の軸表示を追加 -->
+            <visual name="debug_x_axis">
+                <origin xyz="0.02 0 0" rpy="0 ${radians(90)} 0"/>
+                <geometry>
+                    <cylinder radius="0.002" length="0.04"/>
+                </geometry>
+                <material name="debug_red">
+                    <color rgba="1.0 0.0 0.0 1.0"/>
+                </material>
+            </visual>
+            <visual name="debug_y_axis">
+                <origin xyz="0 0.02 0" rpy="${radians(90)} 0 0"/>
+                <geometry>
+                    <cylinder radius="0.002" length="0.04"/>
+                </geometry>
+                <material name="debug_green">
+                    <color rgba="0.0 1.0 0.0 1.0"/>
+                </material>
+            </visual>
+            <visual name="debug_z_axis">
+                <origin xyz="0 0 0.02" rpy="0 0 0"/>
+                <geometry>
+                    <cylinder radius="0.002" length="0.04"/>
+                </geometry>
+                <material name="debug_blue">
+                    <color rgba="0.0 0.0 1.0 1.0"/>
+                </material>
+            </visual>
         </link>
         <!-- 脚先（foot_tip）を示す非常に小さなリンク -->
@@ -109,17 +137,45 @@
             <inertial>
                 <origin xyz="0 0 0" rpy="0 0 0"/>
-                <!-- 非常に軽い質量（物理シミュレーションにほとんど影響しない） -->
                 <mass value="0.0001"/>
                 <inertia ixx="0.00001" iyy="0.00001" izz="0.00001" ixy="0.0" iyz="0.0" ixz="0.0"/>
             </inertial>
-            <!-- 小さな視覚マーカー（オプション） -->
-            <visual>
-                <origin xyz="0 0 0" rpy="0 0 0"/>
-                <geometry>
-                    <!-- とても小さな球体マーカー -->
-                    <sphere radius="0.003"/>
+            <!-- X軸（前方向）- 赤色 -->
+            <visual name="x_axis">
+                <origin xyz="0.01 0 0" rpy="0 ${radians(90)} 0"/>
+                <geometry>
+                    <cylinder radius="0.001" length="0.02"/>
                 </geometry>
                 <material name="red">
                     <color rgba="1.0 0.0 0.0 1.0"/>
+                </material>
+            </visual>
+            <!-- Y軸（右方向）- 緑色 -->
+            <visual name="y_axis">
+                <origin xyz="0 0.01 0" rpy="${radians(90)} 0 0"/>
+                <geometry>
+                    <cylinder radius="0.001" length="0.02"/>
+                </geometry>
+                <material name="green">
+                    <color rgba="0.0 1.0 0.0 1.0"/>
+                </material>
+            </visual>
+            <!-- Z軸（上方向）- 青色 -->
+            <visual name="z_axis">
+                <origin xyz="0 0 0.01" rpy="0 0 0"/>
+                <geometry>
+                    <cylinder radius="0.001" length="0.02"/>
+                </geometry>
+                <material name="blue">
+                    <color rgba="0.0 0.0 1.0 1.0"/>
+                </material>
+            </visual>
+            <!-- 座標原点 - 白色 -->
+            <visual name="origin">
+                <origin xyz="0 0 0" rpy="0 0 0"/>
+                <geometry>
+                    <sphere radius="0.003"/>
+                </geometry>
+                <material name="white">
+                    <color rgba="1.0 1.0 1.0 1.0"/>
                 </material>
             </visual>
@@ -156,5 +212,5 @@
         <joint name="limb${limb_id}_foot_joint" type="fixed">
             <!-- tibiaのSTLモデルの先端までの距離を設定 -->
-            <origin xyz="-0.103 0.0205 -0.00205" rpy="0 0 0"/>
+            <origin xyz="-0.103 0.0205 -0.00205" rpy="${radians(-90)} 0 ${radians(-90)}"/>
             <parent link="limb${limb_id}_link6"/>
             <child link="limb${limb_id}_foot_tip"/>

File: model/urdf/hexa_leg_pod.urdf (robot description, URDF)
Before this commit: robot hexa_leg_pod, 32 links, 31 joints
Links:
- link limb0_foot_tip: geometry visual cylinder length=0.02 radius=0.001; visual cylinder length=0.02 radius=0.001
- link limb0_link6: geometry collision mesh filename=package://dual_leg_controller/model/meshes/link3_1.stl scale=0.001 0.001 0.001; visual cylinder length=0.04 radius=0.002
- link limb1_foot_tip: geometry visual cylinder length=0.02 radius=0.001; visual cylinder length=0.02 radius=0.001
- link limb1_link6: geometry collision mesh filename=package://dual_leg_controller/model/meshes/link3_1.stl scale=0.001 0.001 0.001; visual cylinder length=0.04 radius=0.002
- link limb2_foot_tip: geometry visual cylinder length=0.02 radius=0.001; visual cylinder length=0.02 radius=0.001
- link limb2_link6: geometry collision mesh filename=package://dual_leg_controller/model/meshes/link3_1.stl scale=0.001 0.001 0.001; visual cylinder length=0.04 radius=0.002
- link limb3_foot_tip: geometry visual cylinder length=0.02 radius=0.001; visual cylinder length=0.02 radius=0.001
- link limb3_link6: geometry collision mesh filename=package://dual_leg_controller/model/meshes/link3_1.stl scale=0.001 0.001 0.001; visual cylinder length=0.04 radius=0.002
- link limb4_foot_tip: geometry visual cylinder length=0.02 radius=0.001; visual cylinder length=0.02 radius=0.001
- link limb4_link6: geometry collision mesh filename=package://dual_leg_controller/model/meshes/link3_1.stl scale=0.001 0.001 0.001; visual cylinder length=0.04 radius=0.002
- link limb5_foot_tip: geometry visual cylinder length=0.02 radius=0.001; visual cylinder length=0.02 radius=0.001
- link limb5_link6: geometry collision mesh filename=package://dual_leg_controller/model/meshes/link3_1.stl scale=0.001 0.001 0.001; visual cylinder length=0.04 radius=0.002
Joints:
- joint limb0_foot_joint: origin xyz=-0.103 0.0205 -0.00205 rpy=0 0 0 -> xyz=-0.103 0.0205 -0.00205 rpy=-1.5707963267948966 0 -1.5707963267948966
- joint limb1_foot_joint: origin xyz=-0.103 0.0205 -0.00205 rpy=0 0 0 -> xyz=-0.103 0.0205 -0.00205 rpy=-1.5707963267948966 0 -1.5707963267948966
- joint limb2_foot_joint: origin xyz=-0.103 0.0205 -0.00205 rpy=0 0 0 -> xyz=-0.103 0.0205 -0.00205 rpy=-1.5707963267948966 0 -1.5707963267948966
- joint limb3_foot_joint: origin xyz=-0.103 0.0205 -0.00205 rpy=0 0 0 -> xyz=-0.103 0.0205 -0.00205 rpy=-1.5707963267948966 0 -1.5707963267948966
- joint limb4_foot_joint: origin xyz=-0.103 0.0205 -0.00205 rpy=0 0 0 -> xyz=-0.103 0.0205 -0.00205 rpy=-1.5707963267948966 0 -1.5707963267948966
- joint limb5_foot_joint: origin xyz=-0.103 0.0205 -0.00205 rpy=0 0 0 -> xyz=-0.103 0.0205 -0.00205 rpy=-1.5707963267948966 0 -1.5707963267948966

Commit message: [modify]modify programs of xacro "multileg"

File: model/urdf/hexa_leg.xacro (robot description, xacro)
@@ -2,5 +2,5 @@
 <robot name = "hexa_leg_pod" xmlns:xacro = "http://www.ros.org/wiki/xacro">
     <!-- include -->
-    <xacro:include filename="$(find multileg)/urdf/materials.xacro" />
+    <xacro:include filename="$(find dual_leg_controller)/model/urdf/materials.xacro" />
     <!--Setting property-->
     <xacro:property name="motor_height" value="0.02" /> <!--motorを下げる高さ[m]-->
@@ -217,34 +217,34 @@
         </joint>
         <!-- トランスミッション -->
-    <transmission name="trans${limb_id}_1">
-        <type>transmission_interface/SimpleTransmission</type>
-        <joint name="limb${limb_id}_joint1">
-        <hardwareInterface>hardware_interface/EffortJointInterface</hardwareInterface>
-        </joint>
-        <actuator name="motor${limb_id}_1">
-        <hardwareInterface>hardware_interface/EffortJointInterface</hardwareInterface>
-        <mechanicalReduction>1</mechanicalReduction>
-        </actuator>
-    </transmission>
-    <transmission name="trans${limb_id}_2">
-        <type>transmission_interface/SimpleTransmission</type>
-        <joint name="limb${limb_id}_joint2">
-        <hardwareInterface>hardware_interface/EffortJointInterface</hardwareInterface>
-        </joint>
-        <actuator name="motor${limb_id}_2">
-        <hardwareInterface>hardware_interface/EffortJointInterface</hardwareInterface>
-        <mechanicalReduction>1</mechanicalReduction>
-        </actuator>
-    </transmission>
-    <transmission name="trans${limb_id}_3">
-        <type>transmission_interface/SimpleTransmission</type>
-        <joint name="limb${limb_id}_joint3">
-        <hardwareInterface>hardware_interface/EffortJointInterface</hardwareInterface>
-        </joint>
-        <actuator name="motor${limb_id}_3">
-        <hardwareInterface>hardware_interface/EffortJointInterface</hardwareInterface>
-        <mechanicalReduction>1</mechanicalReduction>
-        </actuator>
-    </transmission>
+        <transmission name="trans${limb_id}_1">
+            <type>transmission_interface/SimpleTransmission</type>
+            <joint name="limb${limb_id}_joint1">
+            <hardwareInterface>hardware_interface/EffortJointInterface</hardwareInterface>
+            </joint>
+            <actuator name="motor${limb_id}_1">
+            <hardwareInterface>hardware_interface/EffortJointInterface</hardwareInterface>
+            <mechanicalReduction>1</mechanicalReduction>
+            </actuator>
+        </transmission>
+        <transmission name="trans${limb_id}_2">
+            <type>transmission_interface/SimpleTransmission</type>
+            <joint name="limb${limb_id}_joint2">
+            <hardwareInterface>hardware_interface/EffortJointInterface</hardwareInterface>
+            </joint>
+            <actuator name="motor${limb_id}_2">
+            <hardwareInterface>hardware_interface/EffortJointInterface</hardwareInterface>
+            <mechanicalReduction>1</mechanicalReduction>
+            </actuator>
+        </transmission>
+        <transmission name="trans${limb_id}_3">
+            <type>transmission_interface/SimpleTransmission</type>
+            <joint name="limb${limb_id}_joint3">
+            <hardwareInterface>hardware_interface/EffortJointInterface</hardwareInterface>
+            </joint>
+            <actuator name="motor${limb_id}_3">
+            <hardwareInterface>hardware_interface/EffortJointInterface</hardwareInterface>
+            <mechanicalReduction>1</mechanicalReduction>
+            </actuator>
+        </transmission>
     </xacro:macro>
     <joint name = "body_joint" type="fixed">
@@ -275,4 +275,5 @@
         </collision>
     </link>
+    <!-- 6脚のマクロ呼び出し -->
     <xacro:limb_macro limb_id="0" arc="0"/>
     <xacro:limb_macro limb_id="1" arc="60"/>
@@ -283,5 +284,5 @@
     <gazebo>
         <plugin name="gazebo_ros_control" filename="libgazebo_ros_control.so">
-        <robotNamespace>/multileg</robotNamespace>
+        <robotNamespace>/hexa_leg</robotNamespace>
         </plugin>
     </gazebo>
